File: PCB/PCB.kicad_pcb (KiCad board)
At the start: 2 copper layers, 97.8 x 74.9 mm, 32 parts, among them J1 SMA, J2 12v (Max 18v), Q1 BS170, Q2 BS170, Q3 BS170, U1 Pico, U3 74ACT244, U4 uSDX mOnO Band_MODULE, U5 CDIL_7805_TO220

Commit message: PCB v2 - minor tweaks
Parts:
- removed J2: 12v (Max 18v), Connector_PinHeader_2.54mm:PinHeader_1x02_P2.54mm_Vertical
- added Power1: DC-005 (Barrel Jack), footprints:XKB_DC-005-5A-2.0_Modded, F.Cu at (100.8, 46.5)
- added TP1: TestPoint, TestPoint:TestPoint_THTPad_2.0x2.0mm_Drill1.0mm, F.Cu at (168.1, 77.5)
- Q1, Q2, Q3: footprint Package_TO_SOT_THT:TO-92_Inline -> Package_TO_SOT_THT:TO-92_HandSolder
- moved H2 1.08 mm to (180.1, 48.0)
- moved Q2 0.30 mm to (175.3, 67.5)
- moved H3 0.20 mm to (89.8, 115.6)
- moved Q1 0.20 mm to (175.3, 74.3)
- moved Q3 0.18 mm to (175.3, 60.7)
Routing:
- net TD_IN: track 46.1 -> 47.7 mm
- net Net-(C22-Pad1): track 40.8 -> 39.8 mm
- net Net-(D9-Pad2): track 6.78 -> 5.92 mm
- net GND: vias 166 -> 170
