File: PCB/PCB.kicad_sch (KiCad schematic)
At the start: 32 parts, among them J1 SMA, J2 12v (Max 18v), Q1 BS170, Q2 BS170, Q3 BS170, U1 Pico, U3 74ACT244, U4 uSDX mOnO Band_MODULE, U5 CDIL_7805_TO220

Commit message: PCB v2 - minor tweaks
Parts:
- removed J2: 12v (Max 18v), Connector_PinHeader_2.54mm:PinHeader_1x02_P2.54mm_Vertical, symbol Connector_Generic:Conn_01x02
- added Power1: DC-005 (Barrel Jack), footprints:XKB_DC-005-5A-2.0_Modded, symbol Connector:Barrel_Jack_Switch
- added TP1: TestPoint, TestPoint:TestPoint_THTPad_2.0x2.0mm_Drill1.0mm, symbol Connector:TestPoint
- Q1, Q2, Q3: footprint Package_TO_SOT_THT:TO-92_Inline -> Package_TO_SOT_THT:TO-92_HandSolder
Connections:
- net GND: now also Power1.2
- net at C22.1, D6.1 (K), Q1.2 (G)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: now also TP1.1
- net at D9.2 (A): now also Power1.1
- no-connect marks 40 -> 41
Changed lines of the file:
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@@
   (junction (at 287.401 113.792) (diameter 0) (color 0 0 0 0)
+  )
+  (junction (at 212.3948 160.782) (diameter 0) (color 0 0 0 0)
   )
   (junction (at 259.842 156.972) (diameter 0) (color 0 0 0 0)
@@
   (no_connect (at 91.059 148.336))
   (no_connect (at 91.059 145.796))
+  (no_connect (at 371.1448 135.382))
   (no_connect (at 91.059 117.856))
   (no_connect (at 91.059 122.936))
@@
     (stroke (width 0) (type default) (color 0 0 0 0))
   )
-  (wire (pts (xy 209.931 160.782) (xy 222.631 160.782))
+  (wire (pts (xy 209.931 160.782) (xy 212.3948 160.782))
     (stroke (width 0) (type default) (color 0 0 0 0))
   )
@@
     (stroke (width 0) (type default) (color 0 0 0 0))
   )
-  (wire (pts (xy 366.141 132.842) (xy 371.094 132.842))
+  (wire (pts (xy 366.141 132.842) (xy 371.1448 132.842))
     (stroke (width 0) (type default) (color 0 0 0 0))
   )
@@
     (stroke (width 0) (type default) (color 0 0 0 0))
   )
+  (wire (pts (xy 212.3948 160.782) (xy 222.631 160.782))
+    (stroke (width 0) (type default) (color 0 0 0 0))
+  )
   (wire (pts (xy 283.591 107.442) (xy 283.591 113.792))
     (stroke (width 0) (type default) (color 0 0 0 0))
@@
     (stroke (width 0) (type default) (color 0 0 0 0))
   )
-  (wire (pts (xy 371.094 135.382) (xy 371.094 144.272))
-    (stroke (width 0) (type default) (color 0 0 0 0))
-  )
   (wire (pts (xy 173.101 116.332) (xy 183.261 116.332))
     (stroke (width 0) (type default) (color 0 0 0 0))
@@
   )
   (wire (pts (xy 55.499 117.856) (xy 47.498 117.856))
+    (stroke (width 0) (type default) (color 0 0 0 0))
+  )
+  (wire (pts (xy 212.3948 160.0708) (xy 212.3948 160.782))
     (stroke (width 0) (type default) (color 0 0 0 0))
   )
@@
     )
     (pin "1")
+  )
+  (symbol (lib_id "Connector:Barrel_Jack_Switch") (at 378.7648 135.382 0) (mirror y) (unit 1)
+    (in_bom yes) (on_board yes)
+    (property "Reference" "Power1" (id 0) (at 385.1148 134.1119 0)
+      (effects (font (size 1.27 1.27)) (justify right))
+    )
+    (property "Value" "DC-005 (Barrel Jack)" (id 1) (at 385.1148 136.6519 0)
+      (effects (font (size 1.27 1.27)) (justify right))
+    )
+    (property "Footprint" "footprints:XKB_DC-005-5A-2.0_Modded" (id 2) (at 377.4948 136.398 0)
+      (effects (font (size 1.27 1.27)) hide)
+    )
+    (property "Datasheet" "~" (id 3) (at 377.4948 136.398 0)
+      (effects (font (size 1.27 1.27)) hide)
+    )
+    (pin "1")
+    (pin "2")
+    (pin "3")
   )
   (symbol (lib_id "MCU_RaspberryPi_and_Boards:Pico") (at 73.279 134.366 0) (unit 1)
@@
       (effects (font (size 1.27 1.27)) (justify left))
     )
-    (property "Footprint" "Package_TO_SOT_THT:TO-92_Inline" (id 2) (at 232.791 179.197 0)
+    (property "Footprint" "Package_TO_SOT_THT:TO-92_HandSolder" (id 2) (at 232.791 179.197 0)
       (effects (font (size 1.27 1.27) italic) (justify left) hide)
     )
@@
     (pin "2")
   )
-  (symbol (lib_id "power:GND") (at 371.094 144.272 0) (unit 1)
-    (in_bom yes) (on_board yes)
-    (property "Reference" "#PWR0112" (id 0) (at 371.094 149.352 0)
-      (effects (font (size 1.27 1.27)) hide)
-    )
-    (property "Value" "GNDPWR" (id 1) (at 371.1956 148.1836 0))
-    (property "Footprint" "" (id 2) (at 371.094 144.272 0)
-      (effects (font (size 1.27 1.27)) hide)
-    )
-    (property "Datasheet" "" (id 3) (at 371.094 144.272 0)
+  (symbol (lib_id "power:GND") (at 371.1448 137.922 0) (unit 1)
+    (in_bom yes) (on_board yes)
+    (property "Reference" "#PWR0112" (id 0) (at 371.1448 143.002 0)
+      (effects (font (size 1.27 1.27)) hide)
+    )
+    (property "Value" "GNDPWR" (id 1) (at 371.2464 141.8336 0))
+    (property "Footprint" "" (id 2) (at 371.1448 137.922 0)
+      (effects (font (size 1.27 1.27)) hide)
+    )
+    (property "Datasheet" "" (id 3) (at 371.1448 137.922 0)
       (effects (font (size 1.27 1.27)) hide)
     )
@@
     (pin "1")
   )
+  (symbol (lib_id "Connector:TestPoint") (at 212.3948 160.0708 0) (unit 1)
+    (in_bom yes) (on_board yes)
+    (property "Reference" "TP1" (id 0) (at 213.868 157.0736 0)
+      (effects (font (size 1.27 1.27)) (justify left))
+    )
+    (property "Value" "TestPoint" (id 1) (at 211.5058 154.2288 0)
+      (effects (font (size 1.27 1.27)) (justify left))
+    )
+    (property "Footprint" "TestPoint:TestPoint_THTPad_2.0x2.0mm_Drill1.0mm" (id 2) (at 217.4748 160.0708 0)
+      (effects (font (size 1.27 1.27)) hide)
+    )
+    (property "Datasheet" "~" (id 3) (at 217.4748 160.0708 0)
+      (effects (font (size 1.27 1.27)) hide)
+    )
+    (pin "1")
+  )
   (symbol (lib_id "power:GND") (at 102.9208 123.6472 0) (unit 1)
     (in_bom yes) (on_board yes) (fields_autoplaced)
@@
     (pin "2")
   )
-  (symbol (lib_id "Connector_Generic:Conn_01x02") (at 376.174 132.842 0) (unit 1)
-    (in_bom yes) (on_board yes) (fields_autoplaced)
-    (property "Reference" "J2" (id 0) (at 378.841 132.8419 0)
-      (effects (font (size 1.27 1.27)) (justify left))
-    )
-    (property "Value" "12v (Max 18v)" (id 1) (at 378.841 135.3819 0)
-      (effects (font (size 1.27 1.27)) (justify left))
-    )
-    (property "Footprint" "Connector_PinHeader_2.54mm:PinHeader_1x02_P2.54mm_Vertical" (id 2) (at 376.174 132.842 0)
-      (effects (font (size 1.27 1.27)) hide)
-    )
-    (property "Datasheet" "~" (id 3) (at 376.174 132.842 0)
-      (effects (font (size 1.27 1.27)) hide)
-    )
-    (pin "1")
-    (pin "2")
-  )
   (symbol (lib_id "power:PWR_FLAG") (at 346.964 159.766 0) (unit 1)
     (in_bom yes) (on_board yes) (fields_autoplaced)
@@
       (effects (font (size 1.27 1.27)) (justify left))
     )
-    (property "Footprint" "Package_TO_SOT_THT:TO-92_Inline" (id 2) (at 232.791 148.717 0)
+    (property "Footprint" "Package_TO_SOT_THT:TO-92_HandSolder" (id 2) (at 232.791 148.717 0)
       (effects (font (size 1.27 1.27) italic) (justify left) hide)
     )
@@
       (effects (font (size 1.27 1.27)) (justify left))
     )
-    (property "Footprint" "Package_TO_SOT_THT:TO-92_Inline" (id 2) (at 232.791 163.957 0)
+    (property "Footprint" "Package_TO_SOT_THT:TO-92_HandSolder" (id 2) (at 232.791 163.957 0)
       (effects (font (size 1.27 1.27) italic) (justify left) hide)
     )
@@
       (reference "J1") (unit 1) (value "SMA") (footprint "Connector_Coaxial:SMA_Samtec_SMA-J-P-X-ST-EM1_EdgeMount")
     )
-    (path "/c92065e0-a3b6-4592-ba10-d1c597411a61"
-      (reference "J2") (unit 1) (value "12v (Max 18v)") (footprint "Connector_PinHeader_2.54mm:PinHeader_1x02_P2.54mm_Vertical")
+    (path "/02f6e829-e953-4ce6-b3db-22bd213d1390"
+      (reference "Power1") (unit 1) (value "DC-005 (Barrel Jack)") (footprint "footprints:XKB_DC-005-5A-2.0_Modded")
     )
     (path "/d072b2ff-e457-4581-b972-8d4dfc339474"
-      (reference "Q1") (unit 1) (value "BS170") (footprint "Package_TO_SOT_THT:TO-92_Inline")
+      (reference "Q1") (unit 1) (value "BS170") (footprint "Package_TO_SOT_THT:TO-92_HandSolder")
     )
     (path "/f64d978c-deed-430b-9842-57afc3d5f7af"
-      (reference "Q2") (unit 1) (value "BS170") (footprint "Package_TO_SOT_THT:TO-92_Inline")
+      (reference "Q2") (unit 1) (value "BS170") (footprint "Package_TO_SOT_THT:TO-92_HandSolder")
     )
     (path "/365ff446-d4b1-41db-bd77-58cd44186b6c"
-      (reference "Q3") (unit 1) (value "BS170") (footprint "Package_TO_SOT_THT:TO-92_Inline")
+      (reference "Q3") (unit 1) (value "BS170") (footprint "Package_TO_SOT_THT:TO-92_HandSolder")
     )
     (path "/00000000-0000-0000-0000-000061d8a8b9"
       (reference "R12") (unit 1) (value "2.7k") (footprint "Resistor_THT:R_Axial_DIN0204_L3.6mm_D1.6mm_P1.90mm_Vertical")
     )
+    (path "/63428fa2-103d-4212-9362-9ae582df28e5"
+      (reference "TP1") (unit 1) (value "TestPoint") (footprint "TestPoint:TestPoint_THTPad_2.0x2.0mm_Drill1.0mm")
+    )
     (path "/00000000-0000-0000-0000-00005ef2b443"
